Commit message: small

File: minirover/urdf/gopigo3.urdf.xacro (robot description, xacro)
@@ -48,5 +48,5 @@
       <origin xyz="0.024 0.097 -0.038" rpy="0 0 0"/>
       <geometry>
-        <mesh filename="package://gopigo3_description/meshes/GoPiGo3_Body.stl" scale="${CADscale} ${CADscale} ${CADscale}"/>
+        <mesh filename="package://minirover/meshes/GoPiGo3_Body.stl" scale="${CADscale} ${CADscale} ${CADscale}"/>
       </geometry>
       <material name="blue"/>
@@ -67,5 +67,5 @@
       <origin xyz="-0.195 -0.173 -0.029" rpy="0 0 0"/>
       <geometry>
-        <mesh filename="package://gopigo3_description/meshes/GoPiGo3_Wheel.stl" scale="0.001 0.001 0.001"/>
+        <mesh filename="package://minirover/meshes/GoPiGo3_Wheel.stl" scale="0.001 0.001 0.001"/>
       </geometry>
       <material name="black"/>
@@ -99,5 +99,5 @@
       <origin xyz="-0.195 -0.173 -0.029" rpy="0 0 0"/>
       <geometry>
-        <mesh filename="package://gopigo3_description/meshes/GoPiGo3_Wheel.stl" scale="0.001 0.001 0.001"/>
+        <mesh filename="package://minirover/meshes/GoPiGo3_Wheel.stl" scale="0.001 0.001 0.001"/>
       </geometry>
       <material name="black"/>
@@ -179,5 +179,5 @@
         <origin xyz="0 0 0" rpy="1.57 0 1.57"/>
         <geometry>
-          <mesh filename="package://gopigo3_description/meshes/sensors/IR_Sensor_Sharp_GP2Y_solid.stl" scale="0.001 0.001 0.001"/>
+          <mesh filename="package://minirover/meshes/sensors/IR_Sensor_Sharp_GP2Y_solid.stl" scale="0.001 0.001 0.001"/>
         </geometry>
         <material name="red"/>
@@ -200,6 +200,6 @@
         <origin xyz="0 0 0.0" rpy="0 0 0"/>
         <geometry>
-          <mesh filename="package://gopigo3_description/meshes/sensors/X4.stl" scale="0.001 0.001 0.001"/>
-          <!--LDS** mesh filename="package://gopigo3_description/meshes/sensors/lds.stl" scale="0.001 0.001 0.001"/-->
+          <mesh filename="package://minirover/meshes/sensors/X4.stl" scale="0.001 0.001 0.001"/>
+          <!--LDS** mesh filename="package://minirover/meshes/sensors/lds.stl" scale="0.001 0.001 0.001"/-->
         </geometry>
         <material name="orange"/>
@@ -231,5 +231,5 @@
         <origin xyz="0.005 0.000 0.013" rpy="0 1.570795 0" />
         <geometry>
-            <mesh filename="package://gopigo3_description/meshes/sensors/piCamera.stl" scale="0.00125 0.00125 0.00125"/>
+            <mesh filename="package://minirover/meshes/sensors/piCamera.stl" scale="0.00125 0.00125 0.00125"/>
         </geometry>
         <material name="yellow"/>

Commit message: small

File: minirover/urdf/gopigo3.urdf.xacro (robot description, xacro)
@@ -193,5 +193,5 @@
       <parent link="base_link"/>
       <child link="base_scan"/>
-      <origin xyz="-0.02 0 0.105" rpy="0 0 -1.6"/>
+      <origin xyz="-0.02 0 0.105" rpy="0 0 0"/>
       <!--LDS** origin xyz="-0.02 0 0.07" rpy="0 0 -1.6"/-->
     </joint>

Commit message: small

File: minirover/urdf/gopigo3.urdf.xacro (robot description, xacro)
@@ -13,6 +13,6 @@
   <link name="base_footprint"/>
   <joint name="base_joint" type="fixed">
-    <parent link="base_footprint"/>
-    <child link="base_link"/>
+    <child link="base_footprint"/>
+    <parent link="base_link"/>
     <!-- base_link is placed at the center of gravity of GoPiGo3 body -->
     <origin xyz="0 0 0.075" rpy="0 0 0"/>

Commit message: small

File: minirover/urdf/gopigo3.urdf.xacro (robot description, xacro)
@@ -13,6 +13,6 @@
   <link name="base_footprint"/>
   <joint name="base_joint" type="fixed">
-    <child link="base_footprint"/>
-    <parent link="base_link"/>
+    <parent link="base_footprint"/>
+    <child link="base_link"/>
     <!-- base_link is placed at the center of gravity of GoPiGo3 body -->
     <origin xyz="0 0 0.075" rpy="0 0 0"/>
