Commit message: small change

File: minirover/urdf/minirover.urdf.xacro (robot description, xacro)
@@ -37,5 +37,5 @@
   </link>
 <!-- ============  'base_link_cad' is the solid model of robot body ====== -->
-  <joint name="base_joint_cad" type="fixed">
+  <!-- <joint name="base_joint_cad" type="fixed">
     <parent link="base_footprint"/>
     <child link="base_link_cad"/>
@@ -43,4 +43,5 @@
     <origin xyz="0 0 0.033" rpy="0 0 -4.71"/>
   </joint>
+ -->
   <link name="base_link_cad">
     <visual>

Commit message: small change

File: minirover/urdf/minirover.urdf.xacro (robot description, xacro)
@@ -37,11 +37,10 @@
   </link>
 <!-- ============  'base_link_cad' is the solid model of robot body ====== -->
-  <!-- <joint name="base_joint_cad" type="fixed">
-    <parent link="base_footprint"/>
-    <child link="base_link_cad"/>
+  <!-- <joint name="base_joint_cad" type="fixed"> -->
+    <!-- <parent link="base_footprint"/> -->
+    <!-- <child link="base_link_cad"/> -->
     <!-- CAD of body of GoPiGo3 has its reference coordinate system at the center of the wheels shaft -->
-    <origin xyz="0 0 0.033" rpy="0 0 -4.71"/>
-  </joint>
- -->
+    <!-- <origin xyz="0 0 0.033" rpy="0 0 -4.71"/> -->
+  <!-- </joint> -->
   <link name="base_link_cad">
     <visual>

Commit message: small change

File: minirover/urdf/minirover.urdf.xacro (robot description, xacro)
@@ -37,10 +37,10 @@
   </link>
 <!-- ============  'base_link_cad' is the solid model of robot body ====== -->
-  <!-- <joint name="base_joint_cad" type="fixed"> -->
-    <!-- <parent link="base_footprint"/> -->
-    <!-- <child link="base_link_cad"/> -->
+  <joint name="base_joint_cad" type="fixed">
+    <parent link="base_footprint"/>
+    <child link="base_link_cad"/>
     <!-- CAD of body of GoPiGo3 has its reference coordinate system at the center of the wheels shaft -->
-    <!-- <origin xyz="0 0 0.033" rpy="0 0 -4.71"/> -->
-  <!-- </joint> -->
+    <origin xyz="0 0 0.033" rpy="0 0 0"/>
+  </joint>
   <link name="base_link_cad">
     <visual>

Commit message: small change

File: minirover/urdf/minirover.urdf.xacro (robot description, xacro)
@@ -41,5 +41,5 @@
     <child link="base_link_cad"/>
     <!-- CAD of body of GoPiGo3 has its reference coordinate system at the center of the wheels shaft -->
-    <origin xyz="0 0 0.033" rpy="0 0 0"/>
+    <origin xyz="0 0 0.033" rpy="0 0 1.5707963268"/>
   </joint>
   <link name="base_link_cad">
