Commit message: small change

File: minirover/urdf/minirover1.urdf (robot description, URDF)
Before this commit: robot gopigo, 2 links, 1 joints
Links:
- link porch_link: geometry visual box size=0.12 0.11 0.005

Commit message: small change

File: minirover/urdf/minirover1.urdf (robot description, URDF)
Before this commit: robot gopigo, 2 links, 1 joints
Joints:
- joint porch_link: origin xyz=0 0.0 0.05 rpy=0 0 0 -> xyz=0.08 0.0 0.05 rpy=0 0 0

Commit message: small change

File: minirover/urdf/minirover1.urdf (robot description, URDF)
Before this commit: robot gopigo, 2 links, 1 joints
Joints:
- joint porch_link: origin xyz=0.08 0.0 0.05 rpy=0 0 0 -> xyz=0.04 0.0 0.05 rpy=0 0 0
