Commit message: small change

File: minirover/urdf/minirover.urdf (robot description, URDF)
Before this commit: robot gopigo, 3 links, 2 joints
Links:
- link left_wheel: geometry collision cylinder length=0.02 radius=0.05; visual cylinder length=0.02 radius=0.05
- link right_wheel: geometry collision cylinder length=0.02 radius=0.05; visual cylinder length=0.02 radius=0.05

Commit message: small change

File: minirover/urdf/minirover.urdf (robot description, URDF)
Before this commit: robot gopigo, 3 links, 2 joints
Joints:
- joint joint_left_wheel: origin xyz=0 0.30 0 rpy=0 0 0 -> xyz=0 0.075 0 rpy=0 0 0
- joint joint_right_wheel: origin xyz=0 -0.30 0 rpy=0 0 0 -> xyz=0 -0.075 0 rpy=0 0 0

Commit message: mr_description

File: minirover/urdf/minirover.urdf (robot description, URDF)
Before this commit: robot gopigo, 2 links, 1 joints
Links:
- added link left_wheel; visual cylinder length=0.01 radius=0.03
- added link right_wheel; visual cylinder length=0.01 radius=0.03
Joints:
- added joint left_wheel_joint: type continuous, parent base_link, child left_wheel, origin xyz=0 -0 0 rpy=0 0 0, axis 0 1 0
- added joint right_wheel_joint: type continuous, parent base_link, child right_wheel, origin xyz=0 -0.30 0 rpy=0 0 0, axis 0 1 0

Commit message: mr_description

File: minirover/urdf/minirover.urdf (robot description, URDF)
Before this commit: robot gopigo, 4 links, 3 joints
Joints:
- joint left_wheel_joint: origin xyz=0 -0 0 rpy=0 0 0 -> xyz=0 0.30 0 rpy=0 0 0

Commit message: mr_description

File: minirover/urdf/minirover.urdf (robot description, URDF)
Before this commit: robot gopigo, 4 links, 3 joints
Joints:
- joint right_wheel_joint: origin xyz=0 -0.30 0 rpy=0 0 0 -> xyz=0 -0.30 0 rpy=1.570795 0 0

Commit message: mr_description

File: minirover/urdf/minirover.urdf (robot description, URDF)
Before this commit: robot gopigo, 4 links, 3 joints
Joints:
- joint left_wheel_joint: origin xyz=0 0.30 0 rpy=0 0 0 -> xyz=0 0.05 0 rpy=0 0 0
- joint right_wheel_joint: origin xyz=0 -0.30 0 rpy=1.570795 0 0 -> xyz=0 -0.05 0 rpy=0 0 0

Commit message: mr_description

File: minirover/urdf/minirover.urdf (robot description, URDF)
Before this commit: robot gopigo, 4 links, 3 joints
Joints:
- joint left_wheel_joint: origin xyz=0 0.05 0 rpy=0 0 0 -> xyz=0.-08 0.05 0 rpy=0 0 0
- joint right_wheel_joint: origin xyz=0 -0.05 0 rpy=0 0 0 -> xyz=0.08 -0.05 0 rpy=0 0 0

Commit message: mr_description

File: minirover/urdf/minirover.urdf (robot description, URDF)
Before this commit: robot gopigo, 4 links, 3 joints
Joints:
- joint left_wheel_joint: origin xyz=0.-08 0.05 0 rpy=0 0 0 -> xyz=-0.08 0.05 0 rpy=0 0 0

Commit message: mr_description

File: minirover/urdf/minirover.urdf (robot description, URDF)
Before this commit: robot gopigo, 4 links, 3 joints
Links:
- added link battery_link
Joints:
- added joint battery_joint: type fixed, parent base_link, child battery_link
- joint left_wheel_joint: origin xyz=-0.08 0.05 0 rpy=0 0 0 -> xyz=0.02 0.05 0 rpy=0 0 0
- joint right_wheel_joint: origin xyz=0.08 -0.05 0 rpy=0 0 0 -> xyz=0.02 -0.05 0 rpy=0 0 0

Commit message: mr_description

File: minirover/urdf/minirover.urdf (robot description, URDF)
Before this commit: robot gopigo, 5 links, 4 joints
Links:
- link battery_link: geometry visual box size=0.06 0.1 0.015

Commit message: mr_description

File: minirover/urdf/minirover.urdf (robot description, URDF)
Before this commit: robot gopigo, 5 links, 4 joints
Links:
- link battery_link: geometry visual box size=0.06 0.1 0.02
Joints:
- joint battery_joint: origin (none) -> xyz=-0.04 0.05 0 rpy=0 0 0

Commit message: mr_description

File: minirover/urdf/minirover.urdf (robot description, URDF)
Before this commit: robot gopigo, 5 links, 4 joints
Joints:
- joint battery_joint: origin xyz=-0.04 0.05 0 rpy=0 0 0 -> xyz=-0.04 0 0 rpy=0 0 0

Commit message: mr_description

File: minirover/urdf/minirover.urdf (robot description, URDF)
Before this commit: robot gopigo, 5 links, 4 joints
Joints:
- joint battery_joint: origin xyz=-0.04 0 0 rpy=0 0 0 -> xyz=-0.04 0 0.02 rpy=0 0 0

Commit message: mr_description

File: minirover/urdf/minirover.urdf (robot description, URDF)
Before this commit: robot gopigo, 5 links, 4 joints
Joints:
- joint battery_joint: origin xyz=-0.04 0 0.02 rpy=0 0 0 -> xyz=-0.05 0 0.02 rpy=0 0 0

Commit message: small

File: minirover/urdf/minirover.urdf (robot description, URDF)
Before this commit: robot gopigo, 5 links, 4 joints
Joints:
- joint left_wheel_joint: origin xyz=0.02 0.05 0 rpy=0 0 0 -> xyz=0.02 0.06 0 rpy=0 0 0
- joint right_wheel_joint: origin xyz=0.02 -0.05 0 rpy=0 0 0 -> xyz=0.02 -0.06 0 rpy=0 0 0

Commit message: small

File: minirover/urdf/minirover.urdf (robot description, URDF)
Before this commit: robot gopigo, 5 links, 4 joints
Joints:
- joint left_wheel_joint: origin xyz=0.02 0.06 0 rpy=0 0 0 -> xyz=0.02 0.07 0 rpy=0 0 0
- joint right_wheel_joint: origin xyz=0.02 -0.06 0 rpy=0 0 0 -> xyz=0.02 -0.07 0 rpy=0 0 0

Commit message: small

File: minirover/urdf/minirover.urdf (robot description, URDF)
Before this commit: robot gopigo, 5 links, 4 joints
Links:
- added link lidar_link; visual cylinder length=0.06 radius=0.03
Joints:
- added joint lidar_joint: type fixed, parent porch_link, child lidar_link, origin xyz=-0.05 0 0.02 rpy=0 0 0

Commit message: small

File: minirover/urdf/minirover.urdf (robot description, URDF)
Before this commit: robot gopigo, 6 links, 5 joints
Joints:
- joint lidar_joint: origin xyz=-0.05 0 0.02 rpy=0 0 0 -> xyz=0.05 0 -0.02 rpy=0 0 0

Commit message: small

File: minirover/urdf/minirover.urdf (robot description, URDF)
Before this commit: robot gopigo, 6 links, 5 joints
Joints:
- joint lidar_joint: origin xyz=0.05 0 -0.02 rpy=0 0 0 -> xyz=0.05 0 0.002 rpy=0 0 0

Commit message: small

File: minirover/urdf/minirover.urdf (robot description, URDF)
Before this commit: robot gopigo, 6 links, 5 joints
Links:
- added link plate_link; visual box size=0.2 0.11 0.005
- link base_link: geometry 
Joints:
- added joint plate_link: type fixed, parent base_link, child plate_link, origin xyz=0.04 0.0 0.05 rpy=0 0 0
- joint lidar_joint: origin xyz=0.05 0 0.002 rpy=0 0 0 -> xyz=0.00 0 0.03 rpy=0 0 0
- joint porch_link: parent base_link -> plate_link

Commit message: small

File: minirover/urdf/minirover.urdf (robot description, URDF)
Before this commit: robot gopigo, 7 links, 6 joints
Joints:
- joint plate_link: origin xyz=0.04 0.0 0.05 rpy=0 0 0 -> xyz=0.04 0.0 -0.05 rpy=0 0 0

Commit message: small

File: minirover/urdf/minirover.urdf (robot description, URDF)
Before this commit: robot gopigo, 7 links, 6 joints
Joints:
- removed joint plate_link
- removed joint porch_link
- added joint plate_link_joint: type fixed, parent base_link, child plate_link, origin xyz=0.04 0.0 -0.05 rpy=0 0 0
- added joint porch_link_joint: type fixed, parent plate_link, child porch_link, origin xyz=0.04 0.0 0.05 rpy=0 0 0

Commit message: small

File: minirover/urdf/minirover.urdf (robot description, URDF)
Before this commit: robot gopigo, 7 links, 6 joints
Joints:
- joint plate_link_joint: origin xyz=0.04 0.0 -0.05 rpy=0 0 0 -> xyz=0.04 0.0 0.05 rpy=0 0 0

Commit message: small

File: minirover/urdf/minirover.urdf (robot description, URDF)
Before this commit: robot gopigo, 7 links, 6 joints
Joints:
- joint battery_joint: parent base_link -> plate_link
- joint left_wheel_joint: parent base_link -> plate_link
- joint right_wheel_joint: parent base_link -> plate_link

Commit message: small

File: minirover/urdf/minirover.urdf (robot description, URDF)
Before this commit: robot gopigo, 7 links, 6 joints
Links:
- removed link lidar_link
- added link base_scan; visual cylinder length=0.06 radius=0.03
Joints:
- joint lidar_joint: child lidar_link -> base_scan

Commit message: tweaks

File: minirover/urdf/minirover.urdf (robot description, URDF)
Before this commit: robot gopigo, 7 links, 6 joints
Joints:
- joint battery_joint: origin xyz=-0.05 0 0.02 rpy=0 0 0 -> xyz=0.05 0 0.02 rpy=0 0 0
- joint lidar_joint: origin xyz=0.00 0 0.03 rpy=0 0 0 -> xyz=0.05 0 0 rpy=0 0 0

Commit message: rename

File: minirover/urdf/minirover.urdf (robot description, URDF)
Before this commit: robot gopigo, 7 links, 6 joints
Links:
- link base_scan: geometry visual cylinder length=0.055 radius=0.034
- link plate_link: geometry visual box size=0.21 0.09 0.005
- link porch_link: geometry visual box size=0.12 0.105 0.005
Joints:
- joint battery_joint: origin xyz=0.05 0 0.02 rpy=0 0 0 -> xyz=-0.05 0 0.02 rpy=0 0 0
- joint left_wheel_joint: origin xyz=0.02 0.07 0 rpy=0 0 0 -> xyz=0.03 0.07 0 rpy=0 0 0
- joint lidar_joint: origin xyz=0.05 0 0 rpy=0 0 0 -> xyz=-0.02 0 0.03 rpy=0 0 0
- joint plate_link_joint: origin xyz=0.04 0.0 0.05 rpy=0 0 0 -> xyz=-0.0 0.0 0.03 rpy=0 0 0
- joint porch_link_joint: origin xyz=0.04 0.0 0.05 rpy=0 0 0 -> xyz=0.03 0.0 0.05 rpy=0 0 0
- joint right_wheel_joint: origin xyz=0.02 -0.07 0 rpy=0 0 0 -> xyz=0.03 -0.07 0 rpy=0 0 0
