Commit message: updating urdf

File: platform/urdf/platform.urdf (robot description, URDF)
Before this commit: robot bullet, 3 links, 2 joints
Joints:
- joint left_wheel_joint: origin xyz=0 0 0.03 rpy=0 0 0 -> xyz=0 0 -0.03 rpy=0 0 0
- joint right_wheel_joint: origin xyz=0 0 0.03 rpy=0 0 0 -> xyz=0 0 -0.03 rpy=0 0 0
