Commit message: derive all transforms from urd

File: platform/urdf/platform1.urdf (robot description, URDF)
Before this commit: robot platform, 5 links, 4 joints
Joints:
- joint base_link_to_base_footprint: child base_footprint -> base_link; parent base_link -> base_footprint

Commit message: added imu_link to urdf platform1

File: platform/urdf/platform1.urdf (robot description, URDF)
Before this commit: robot platform, 5 links, 4 joints
Links:
- added link imu_link; visual box size=.03 .03 .005
Joints:
- joint base_link_to_scan_link: child scan_link -> imu_link; origin xyz=-0.17 0 0.1 -> xyz=-0.02 0 0.05

Commit message: added imu_link to urdf platform1

File: platform/urdf/platform1.urdf (robot description, URDF)
Before this commit: robot platform, 6 links, 4 joints
Joints:
- added joint base_link_to_imu_link: type fixed, parent base_link, child imu_link, origin xyz=-0.02 0 0.05
- joint base_link_to_scan_link: child imu_link -> scan_link; origin xyz=-0.02 0 0.05 -> xyz=-0.17 0 0.1

Commit message: change sign in urdf

File: platform/urdf/platform1.urdf (robot description, URDF)
Before this commit: robot platform, 6 links, 5 joints
Joints:
- joint base_link_to_base_footprint: origin xyz=0 0 -0.045 -> xyz=0 0 gi0.045

Commit message: change sign in urdf

File: platform/urdf/platform1.urdf (robot description, URDF)
Before this commit: robot platform, 6 links, 5 joints
Joints:
- joint base_link_to_base_footprint: origin xyz=0 0 gi0.045 -> xyz=0 0 0.045

Commit message: latest from paltform2

File: platform/urdf/platform1.urdf (robot description, URDF)
Before this commit: robot platform, 6 links, 5 joints
Joints:
- joint base_link_to_scan_link: origin xyz=-0.17 0 0.1 -> xyz=-0.17 0 0.1 rpy=0 0 3.141
