Commit message: work in progress

File: plat/urdf/platform1.urdf (robot description, URDF)
Before this commit: robot platform, 6 links, 5 joints
Links:
- added link camera_link; visual box size=0.05 0.05 0.05
Joints:
- joint base_link_to_scan_link: child scan_link -> camera_link; origin xyz=-0.17 0 0.1 rpy=0 0 3.141 -> xyz=0.08 0 0.05 rpy=0 0 3.141

Commit message: work in progress

File: plat/urdf/platform1.urdf (robot description, URDF)
Before this commit: robot platform, 7 links, 5 joints
Joints:
- added joint base_link_to_camera_link: type fixed, parent base_link, child camera_link, origin xyz=0.08 0 0.05 rpy=0 0 3.141
- joint base_link_to_scan_link: child camera_link -> scan_link; origin xyz=0.08 0 0.05 rpy=0 0 3.141 -> xyz=-0.17 0 0.1 rpy=0 0 3.141

Commit message: work in progress

File: plat/urdf/platform1.urdf (robot description, URDF)
Before this commit: robot platform, 7 links, 6 joints
Joints:
- removed joint base_link_to_camera_link
- added joint Footprint_to_camera_link: type fixed, parent base_link, child camera_link, origin xyz=0.08 0 0.1 rpy=${-pi/2} 0 ${-pi/2}

Commit message: work in progress

File: plat/urdf/platform1.urdf (robot description, URDF)
Before this commit: robot platform, 7 links, 6 joints
Joints:
- joint Footprint_to_camera_link: parent base_link -> base_footprint
